File: UVTrack - Código.brd (EAGLE design)
At the start: 196.2 x 125.7 mm, 12 parts

Commit message: Arquivos adicionados
Parts:
- removed TINTERRUPTOR_ELETRÔNICO: NPN, Tinkercad:TO92
- added QINTERRUPTOR_ELETRÔNICO: TIP120_TO220-V, Tinkercad:TO220V
Connections:
- removed net TINTERRUPTOR_ELETRÔNICO_B: RBASE_DO_INTERRUPTOR_(TRANSISTOR_NPN).1, TINTERRUPTOR_ELETRÔNICO.2
- new net QINTERRUPTOR_ELETRÔNICO_B: QINTERRUPTOR_ELETRÔNICO.1, RBASE_DO_INTERRUPTOR_(TRANSISTOR_NPN).1
- net MMÓDULO_SIMULADOR_DE_VIBRAÇÃO_-: now also QINTERRUPTOR_ELETRÔNICO.2; no longer TINTERRUPTOR_ELETRÔNICO.1
- net ULILYPAD_VIRTUAL_GND: now also QINTERRUPTOR_ELETRÔNICO.3; no longer TINTERRUPTOR_ELETRÔNICO.3
